File: X14-Conversion.brd (EAGLE design)
At the start: 50.8 x 68.6 mm, 25 parts, among them P1 282837-2, P2 282837-2, P3 282837-2, U1 BUCK,LM2678S-ADJ

Commit message: small adjustments
Parts:
- moved U$3 2.16 mm to (27.8, 5.71)
Routing:
- net 3.3V: track 17.0 -> 20.4 mm
Changed lines of the file:
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@@
 <?xml version="1.0" encoding="utf-8"?>
 <!DOCTYPE eagle SYSTEM "eagle.dtd">
-<eagle version="9.6.2">
+<eagle version="9.5.0">
 <drawing>
 <settings>
@@
 </class>
 </classes>
-<designrules name="477">
+<designrules name="ECE_Senior_Design">
 <description language="de">&lt;b&gt;EAGLE Design Rules&lt;/b&gt;
 &lt;p&gt;
@@
 Einstellungen hier und speichern die Design Rules unter
 einem neuen Namen ab.</description>
-<description language="en">description[de] = &lt;b&gt;EAGLE Design Rules&lt;/b&gt;
-&lt;p&gt;
-Die Standard-Design-Rules sind so gewÃ¤hlt, dass sie fÃ¼r
-die meisten Anwendungen passen. Sollte ihre Platine
-besondere Anforderungen haben, treffen Sie die erforderlichen
-Einstellungen hier und speichern die Design Rules unter
-einem neuen Namen ab.
-description[en] = &lt;b&gt;ECE 402/477 Design Rules Version 2&lt;/b&gt;
+<description language="en">&lt;b&gt;ECE 402/477 Design Rules Version 2&lt;/b&gt;
 &lt;p&gt;
 These are the design rules to use for Purdue University electrical and computer engineering senior design PCBs.
@@
 Please make sure your boards conform to these design rules.
 &lt;/p&gt;
-layerSetup = (1*16)
-mtCopper = 0.0356mm 0.0356mm 0.0356mm 0.0356mm 0.0356mm 0.0356mm 0.0356mm 0.0356mm 0.0356mm 0.0356mm 0.0356mm 0.0356mm 0.0356mm 0.0356mm 0.0356mm 0.0356mm
-mtIsolate = 1.5011mm 0.1499mm 0.2007mm 0.1499mm 0.2007mm 0.1499mm 0.2007mm 0.1499mm 0.2007mm 0.1499mm 0.2007mm 0.1499mm 0.2007mm 0.1499mm 0.2007mm
-mdWireWire = 8mil
-mdWirePad = 8mil
-mdWireVia = 8mil
-mdPadPad = 6mil
-mdPadVia = 8mil
-mdViaVia = 8mil
-mdSmdPad = 6mil
-mdSmdVia = 6mil
-mdSmdSmd = 6mil
-mdViaViaSameLayer = 8mil
-mnLayersViaInSmd = 2
-mdCopperDimension = 15mil
-mdDrill = 8mil
-mdSmdStop = 0mil
-msWidth = 8mil
-msDrill = 13mil
-msMicroVia = 13mil
-msBlindViaRatio = 0.500000
-rvPadTop = 0.250000
-rvPadInner = 0.250000
-rvPadBottom = 0.250000
-rvViaOuter = 0.250000
-rvViaInner = 0.250000
-rvMicroViaOuter = 0.250000
-rvMicroViaInner = 0.250000
-rlMinPadTop = 7mil
-rlMaxPadTop = 20mil
-rlMinPadInner = 7mil
-rlMaxPadInner = 20mil
-rlMinPadBottom = 7mil
-rlMaxPadBottom = 20mil
-rlMinViaOuter = 7mil
-rlMaxViaOuter = 20mil
-rlMinViaInner = 7mil
-rlMaxViaInner = 20mil
-rlMinMicroViaOuter = 4mil
-rlMaxMicroViaOuter = 20mil
-rlMinMicroViaInner = 4mil
-rlMaxMicroViaInner = 20mil
-psTop = -1
-psBottom = -1
-psFirst = -1
-psElongationLong = 100
-psElongationOffset = 100
-mvStopFrame = 1.000000
-mvCreamFrame = 0.000000
-mlMinStopFrame = 3mil
-mlMaxStopFrame = 3mil
-mlMinCreamFrame = 0mil
-mlMaxCreamFrame = 0mil
-mlViaStopLimit = 0mil
-srRoundness = 0.000000
-srMinRoundness = 0mil
-srMaxRoundness = 0mil
-slThermalIsolate = 10mil
-slThermalsForVias = 0
-dpMaxLengthDifference = 10mm
-dpGapFactor = 2.500000
-checkGrid = 0
-checkAngle = 0
-checkFont = 1
-checkRestrict = 1
-useDiameter = 13
-maxErrors = 50
 </description>
 <param name="layerSetup" value="(1*16)"/>
-<param name="mtCopper" value="0.035mm 0.035mm 0.035mm 0.035mm 0.035mm 0.035mm 0.035mm 0.035mm 0.035mm 0.035mm 0.035mm 0.035mm 0.035mm 0.035mm 0.035mm 0.035mm"/>
-<param name="mtIsolate" value="1.5mm 0.15mm 0.2mm 0.15mm 0.2mm 0.15mm 0.2mm 0.15mm 0.2mm 0.15mm 0.2mm 0.15mm 0.2mm 0.15mm 0.2mm"/>
-<param name="mdWireWire" value="6mil"/>
-<param name="mdWirePad" value="6mil"/>
-<param name="mdWireVia" value="6mil"/>
+<param name="mtCopper" value="0.0356mm 0.0356mm 0.0356mm 0.0356mm 0.0356mm 0.0356mm 0.0356mm 0.0356mm 0.0356mm 0.0356mm 0.0356mm 0.0356mm 0.0356mm 0.0356mm 0.0356mm 0.0356mm"/>
+<param name="mtIsolate" value="1.5011mm 0.1499mm 0.2007mm 0.1499mm 0.2007mm 0.1499mm 0.2007mm 0.1499mm 0.2007mm 0.1499mm 0.2007mm 0.1499mm 0.2007mm 0.1499mm 0.2007mm"/>
+<param name="mdWireWire" value="8mil"/>
+<param name="mdWirePad" value="8mil"/>
+<param name="mdWireVia" value="8mil"/>
 <param name="mdPadPad" value="6mil"/>
-<param name="mdPadVia" value="6mil"/>
-<param name="mdViaVia" value="6mil"/>
+<param name="mdPadVia" value="8mil"/>
+<param name="mdViaVia" value="8mil"/>
 <param name="mdSmdPad" value="6mil"/>
 <param name="mdSmdVia" value="6mil"/>
 <param name="mdSmdSmd" value="6mil"/>
-<param name="mdViaViaSameLayer" value="6mil"/>
+<param name="mdViaViaSameLayer" value="8mil"/>
 <param name="mnLayersViaInSmd" value="2"/>
-<param name="mdCopperDimension" value="40mil"/>
-<param name="mdDrill" value="6mil"/>
+<param name="mdCopperDimension" value="15mil"/>
+<param name="mdDrill" value="8mil"/>
 <param name="mdSmdStop" value="0mil"/>
-<param name="msWidth" value="6mil"/>
-<param name="msDrill" value="0.35mm"/>
-<param name="msMicroVia" value="9.99mm"/>
+<param name="msWidth" value="8mil"/>
+<param name="msDrill" value="13mil"/>
+<param name="msMicroVia" value="13mil"/>
 <param name="msBlindViaRatio" value="0.5"/>
 <param name="rvPadTop" value="0.25"/>
@@
 <param name="rvMicroViaOuter" value="0.25"/>
 <param name="rvMicroViaInner" value="0.25"/>
-<param name="rlMinPadTop" value="10mil"/>
+<param name="rlMinPadTop" value="7mil"/>
 <param name="rlMaxPadTop" value="20mil"/>
-<param name="rlMinPadInner" value="10mil"/>
+<param name="rlMinPadInner" value="7mil"/>
 <param name="rlMaxPadInner" value="20mil"/>
-<param name="rlMinPadBottom" value="10mil"/>
+<param name="rlMinPadBottom" value="7mil"/>
 <param name="rlMaxPadBottom" value="20mil"/>
-<param name="rlMinViaOuter" value="8mil"/>
+<param name="rlMinViaOuter" value="7mil"/>
 <param name="rlMaxViaOuter" value="20mil"/>
-<param name="rlMinViaInner" value="8mil"/>
+<param name="rlMinViaInner" value="7mil"/>
 <param name="rlMaxViaInner" value="20mil"/>
 <param name="rlMinMicroViaOuter" value="4mil"/>
@@
 <param name="mvStopFrame" value="1"/>
 <param name="mvCreamFrame" value="0"/>
-<param name="mlMinStopFrame" value="4mil"/>
-<param name="mlMaxStopFrame" value="4mil"/>
+<param name="mlMinStopFrame" value="3mil"/>
+<param name="mlMaxStopFrame" value="3mil"/>
 <param name="mlMinCreamFrame" value="0mil"/>
 <param name="mlMaxCreamFrame" value="0mil"/>
@@
 </element>
 <element name="U$2" library="testpoints" package="3.3V_TESTPOINT" value="3.3V_TESTPOINT" x="44.577" y="16.51" smashed="yes"/>
-<element name="U$3" library="testpoints" package="5.2V_TESTPOINT" value="5.2V_TESTPOINT" x="27.813" y="7.874" smashed="yes"/>
+<element name="U$3" library="testpoints" package="5.2V_TESTPOINT" value="5.2V_TESTPOINT" x="27.813" y="5.715" smashed="yes"/>
 <element name="U$4" library="testpoints" package="12V_TESTPOINT" value="12V_TESTPOINT" x="44.577" y="45.212" smashed="yes"/>
 <element name="U$5" library="testpoints" package="GND_TESTPOINT" value="GND_TESTPOINT" x="30.353" y="64.008" smashed="yes"/>
@@
 <via x="24.257" y="64.008" extent="1-16" drill="0.6"/>
 <via x="30.353" y="59.182" extent="1-16" drill="0.6"/>
-<wire x1="21.209" y1="38.52" x2="21.336" y2="38.52" width="0.254" layer="1"/>
-<wire x1="25.4" y1="38.52" x2="25.273" y2="38.52" width="0.254" layer="1"/>
 <via x="40.894" y="24.638" extent="1-16" drill="0.6"/>
 <via x="46.736" y="24.638" extent="1-16" drill="0.6"/>
-<wire x1="25.4" y1="38.52" x2="25.527" y2="38.52" width="0.254" layer="1"/>
 <contactref element="COUT1" pad="-"/>
 <contactref element="COUT2" pad="-"/>
@@
 <wire x1="25.4" y1="38.354" x2="25.4" y2="37.084" width="0.4064" layer="1"/>
 <via x="25.4" y="37.084" extent="1-16" drill="0.6"/>
-<wire x1="29.2109" y1="40.2209" x2="29.21" y2="40.22" width="0.4064" layer="1"/>
 <wire x1="21.209" y1="38.52" x2="21.209" y2="37.084" width="0.4064" layer="1"/>
 <via x="21.209" y="37.084" extent="1-16" drill="0.6"/>
@@
 <vertex x="29.7688" y="20.59305"/>
 <vertex x="44.6659" y="20.59305"/>
-<vertex x="44.6659" y="11.4808"/>
-<vertex x="37.9984" y="11.4808"/>
+<vertex x="44.6659" y="11.8618"/>
+<vertex x="37.9984" y="11.8618"/>
 <vertex x="37.9984" y="8.2296"/>
 <vertex x="33.5026" y="8.2296"/>
@@
 <vertex x="33.5026" y="8.2296"/>
 <vertex x="37.9984" y="8.2296"/>
-<vertex x="37.9984" y="11.4808"/>
-<vertex x="44.6659" y="11.4808"/>
+<vertex x="37.9984" y="11.8618"/>
+<vertex x="44.6659" y="11.8618"/>
 </polygon>
+<wire x1="9.525" y1="19.304" x2="12.8284" y2="19.304" width="0.762" layer="1"/>
 </signal>
 <signal name="5.2V">
@@
 <vertex x="18.415" y="10.795"/>
 <vertex x="32.6898" y="10.795"/>
-<vertex x="32.6898" y="7.5438"/>
-<vertex x="38.8112" y="7.5438"/>
+<vertex x="32.6898" y="7.2898"/>
+<vertex x="38.8112" y="7.2898"/>
 <vertex x="38.8112" y="10.795"/>
 <vertex x="42.9514" y="10.795"/>
@@
 <vertex x="42.9514" y="10.795"/>
 <vertex x="38.8112" y="10.795"/>
-<vertex x="38.8112" y="7.5438"/>
-<vertex x="32.6898" y="7.5438"/>
+<vertex x="38.8112" y="7.2898"/>
+<vertex x="32.6898" y="7.2898"/>
 <vertex x="32.6898" y="10.795"/>
 <vertex x="28.7655" y="10.795"/>

Commit message: Fix board
Routing:
- net 3.3V: track 20.4 -> 40.3 mm
- net 12V: vias 6 -> 0
- removed copper zone on layer 16, net 12V
Changed lines of the file:
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@@
 <?xml version="1.0" encoding="utf-8"?>
 <!DOCTYPE eagle SYSTEM "eagle.dtd">
-<eagle version="9.5.0">
+<eagle version="9.6.2">
 <drawing>
 <settings>
@@
 <vertex x="44.6659" y="11.8618"/>
 <vertex x="37.9984" y="11.8618"/>
-<vertex x="37.9984" y="8.2296"/>
-<vertex x="33.5026" y="8.2296"/>
-<vertex x="33.5026" y="11.6078"/>
-<vertex x="29.7688" y="11.6078"/>
+<vertex x="37.9984" y="8.1026"/>
+<vertex x="33.5026" y="8.1026"/>
+<vertex x="33.5026" y="11.8618"/>
+<vertex x="29.7688" y="11.8618"/>
 </polygon>
 <wire x1="12.8284" y1="19.304" x2="13.5414125" y2="19.304" width="0.6096" layer="1"/>
 <wire x1="15.0495" y1="18.1728" x2="14.90423125" y2="18.1728" width="0.508" layer="1"/>
-<wire x1="14.90423125" y1="18.1728" x2="13.5414125" y2="19.304" width="0.6096" layer="1"/>
+<wire x1="14.90423125" y1="18.1728" x2="13.5414125" y2="19.304" width="0.762" layer="1"/>
 <wire x1="16.383" y1="18.161" x2="16.3712" y2="18.1728" width="0.508" layer="1"/>
 <wire x1="16.3712" y1="18.1728" x2="15.0495" y2="18.1728" width="0.762" layer="1"/>
@@
 <polygon width="0.508" layer="16" isolate="0.3048">
 <vertex x="44.6659" y="20.59305"/>
-<vertex x="11.8999" y="20.59305"/>
-<vertex x="11.8999" y="11.6078"/>
-<vertex x="33.5026" y="11.6078"/>
-<vertex x="33.5026" y="8.2296"/>
-<vertex x="37.9984" y="8.2296"/>
+<vertex x="29.7688" y="20.59305"/>
+<vertex x="29.7688" y="11.8618"/>
+<vertex x="33.5026" y="11.8618"/>
+<vertex x="33.5026" y="8.1026"/>
+<vertex x="37.9984" y="8.1026"/>
 <vertex x="37.9984" y="11.8618"/>
 <vertex x="44.6659" y="11.8618"/>
 </polygon>
 <wire x1="9.525" y1="19.304" x2="12.8284" y2="19.304" width="0.762" layer="1"/>
+<wire x1="16.383" y1="18.161" x2="30.734" y2="18.161" width="0.762" layer="16"/>
+<wire x1="30.734" y1="18.161" x2="34.671" y2="14.224" width="0.762" layer="16"/>
 </signal>
 <signal name="5.2V">
@@
 <contactref element="CONN" pad="8"/>
 <polygon width="0.508" layer="16" isolate="0.3048">
-<vertex x="18.415" y="10.795"/>
-<vertex x="32.6898" y="10.795"/>
+<vertex x="18.415" y="11.049"/>
+<vertex x="32.6898" y="11.049"/>
 <vertex x="32.6898" y="7.2898"/>
 <vertex x="38.8112" y="7.2898"/>
-<vertex x="38.8112" y="10.795"/>
-<vertex x="42.9514" y="10.795"/>
-<vertex x="42.9514" y="4.953"/>
-<vertex x="18.415" y="4.953"/>
+<vertex x="38.8112" y="11.049"/>
+<vertex x="42.9514" y="11.049"/>
+<vertex x="42.9514" y="5.842"/>
+<vertex x="18.415" y="5.842"/>
 </polygon>
 <contactref element="COUT1" pad="+"/>
@@
 <vertex x="11.963396875" y="20.59178125"/>
 <vertex x="18.415" y="20.59178125"/>
-<vertex x="18.415" y="4.953"/>
-<vertex x="42.9514" y="4.953"/>
-<vertex x="42.9514" y="10.795"/>
-<vertex x="38.8112" y="10.795"/>
+<vertex x="18.415" y="5.842"/>
+<vertex x="42.9514" y="5.842"/>
+<vertex x="42.9514" y="11.049"/>
+<vertex x="38.8112" y="11.049"/>
 <vertex x="38.8112" y="7.2898"/>
 <vertex x="32.6898" y="7.2898"/>
-<vertex x="32.6898" y="10.795"/>
-<vertex x="28.7655" y="10.795"/>
+<vertex x="32.6898" y="11.049"/>
+<vertex x="28.7655" y="11.049"/>
 <vertex x="28.7655" y="36.2077"/>
 </polygon>
@@
 <wire x1="21.844" y1="40.855" x2="21.209" y2="40.22" width="0.762" layer="1"/>
 <wire x1="21.844" y1="40.855" x2="21.844" y2="42.832" width="0.762" layer="1"/>
-<polygon width="0.508" layer="16" isolate="0.3048">
-<vertex x="4.953" y="62.23"/>
-<vertex x="7.493" y="62.23"/>
-<vertex x="7.493" y="57.785"/>
-<vertex x="8.90905" y="56.36895"/>
-<vertex x="18.59915" y="56.36895"/>
-<vertex x="18.59915" y="49.267109375"/>
-<vertex x="30.039309375" y="49.267109375"/>
-<vertex x="30.16885" y="49.39665"/>
-<vertex x="30.16885" y="50.165"/>
-<vertex x="38.5064" y="50.165"/>
-<vertex x="38.5064" y="48.26"/>
-<vertex x="44.6659" y="48.26"/>
-<vertex x="44.6659" y="41.3258"/>
-<vertex x="30.1371" y="41.3258"/>
-<vertex x="30.1371" y="44.7929"/>
-<vertex x="13.7541" y="44.7929"/>
-<vertex x="13.7541" y="50.8381"/>
-<vertex x="7.0739" y="50.8381"/>
-<vertex x="4.953" y="52.959"/>
-</polygon>
 <polygon width="0.508" layer="1" isolate="0.3048">
 <vertex x="4.953" y="62.23"/>
@@
 <vertex x="30.0380375" y="49.2658375"/>
 <vertex x="30.16885" y="49.39665"/>
-<vertex x="30.16885" y="50.165"/>
-<vertex x="38.5064" y="50.165"/>
-<vertex x="38.5064" y="48.26"/>
-<vertex x="44.6659" y="48.26"/>
+<vertex x="30.16885" y="50.1142"/>
+<vertex x="38.5318" y="50.1142"/>
+<vertex x="38.5318" y="48.006"/>
+<vertex x="44.6659" y="48.006"/>
 <vertex x="44.6659" y="41.3258"/>
 <vertex x="30.14345" y="41.3258"/>
@@
 <vertex x="4.953" y="52.959"/>
 </polygon>
-<via x="40.894" y="47.498" extent="1-16" drill="0.6"/>
-<via x="40.894" y="42.672" extent="1-16" drill="0.6"/>
-<via x="34.798" y="47.498" extent="1-16" drill="0.6"/>
-<via x="34.798" y="42.672" extent="1-16" drill="0.6"/>
-<via x="27.94" y="47.498" extent="1-16" drill="0.6"/>
-<via x="21.844" y="47.498" extent="1-16" drill="0.6"/>
 </signal>
 <signal name="SW">

Commit message: fix board
Changed lines of the file:
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@@
 </class>
 </classes>
-<designrules name="ECE_Senior_Design">
+<designrules name="477">
 <description language="de">&lt;b&gt;EAGLE Design Rules&lt;/b&gt;
 &lt;p&gt;
@@
 Einstellungen hier und speichern die Design Rules unter
 einem neuen Namen ab.</description>
-<description language="en">&lt;b&gt;ECE 402/477 Design Rules Version 2&lt;/b&gt;
+<description language="en">description[de] = &lt;b&gt;EAGLE Design Rules&lt;/b&gt;
+&lt;p&gt;
+Die Standard-Design-Rules sind so gewÃ¤hlt, dass sie fÃ¼r
+die meisten Anwendungen passen. Sollte ihre Platine
+besondere Anforderungen haben, treffen Sie die erforderlichen
+Einstellungen hier und speichern die Design Rules unter
+einem neuen Namen ab.
+description[en] = &lt;b&gt;ECE 402/477 Design Rules Version 2&lt;/b&gt;
 &lt;p&gt;
 These are the design rules to use for Purdue University electrical and computer engineering senior design PCBs.
@@
 Please make sure your boards conform to these design rules.
 &lt;/p&gt;
+layerSetup = (1*16)
+mtCopper = 0.0356mm 0.0356mm 0.0356mm 0.0356mm 0.0356mm 0.0356mm 0.0356mm 0.0356mm 0.0356mm 0.0356mm 0.0356mm 0.0356mm 0.0356mm 0.0356mm 0.0356mm 0.0356mm
+mtIsolate = 1.5011mm 0.1499mm 0.2007mm 0.1499mm 0.2007mm 0.1499mm 0.2007mm 0.1499mm 0.2007mm 0.1499mm 0.2007mm 0.1499mm 0.2007mm 0.1499mm 0.2007mm
+mdWireWire = 8mil
+mdWirePad = 8mil
+mdWireVia = 8mil
+mdPadPad = 6mil
+mdPadVia = 8mil
+mdViaVia = 8mil
+mdSmdPad = 6mil
+mdSmdVia = 6mil
+mdSmdSmd = 6mil
+mdViaViaSameLayer = 8mil
+mnLayersViaInSmd = 2
+mdCopperDimension = 15mil
+mdDrill = 8mil
+mdSmdStop = 0mil
+msWidth = 8mil
+msDrill = 13mil
+msMicroVia = 13mil
+msBlindViaRatio = 0.500000
+rvPadTop = 0.250000
+rvPadInner = 0.250000
+rvPadBottom = 0.250000
+rvViaOuter = 0.250000
+rvViaInner = 0.250000
+rvMicroViaOuter = 0.250000
+rvMicroViaInner = 0.250000
+rlMinPadTop = 7mil
+rlMaxPadTop = 20mil
+rlMinPadInner = 7mil
+rlMaxPadInner = 20mil
+rlMinPadBottom = 7mil
+rlMaxPadBottom = 20mil
+rlMinViaOuter = 7mil
+rlMaxViaOuter = 20mil
+rlMinViaInner = 7mil
+rlMaxViaInner = 20mil
+rlMinMicroViaOuter = 4mil
+rlMaxMicroViaOuter = 20mil
+rlMinMicroViaInner = 4mil
+rlMaxMicroViaInner = 20mil
+psTop = -1
+psBottom = -1
+psFirst = -1
+psElongationLong = 100
+psElongationOffset = 100
+mvStopFrame = 1.000000
+mvCreamFrame = 0.000000
+mlMinStopFrame = 3mil
+mlMaxStopFrame = 3mil
+mlMinCreamFrame = 0mil
+mlMaxCreamFrame = 0mil
+mlViaStopLimit = 0mil
+srRoundness = 0.000000
+srMinRoundness = 0mil
+srMaxRoundness = 0mil
+slThermalIsolate = 10mil
+slThermalsForVias = 0
+dpMaxLengthDifference = 10mm
+dpGapFactor = 2.500000
+checkGrid = 0
+checkAngle = 0
+checkFont = 1
+checkRestrict = 1
+useDiameter = 13
+maxErrors = 50
 </description>
 <param name="layerSetup" value="(1*16)"/>
-<param name="mtCopper" value="0.0356mm 0.0356mm 0.0356mm 0.0356mm 0.0356mm 0.0356mm 0.0356mm 0.0356mm 0.0356mm 0.0356mm 0.0356mm 0.0356mm 0.0356mm 0.0356mm 0.0356mm 0.0356mm"/>
-<param name="mtIsolate" value="1.5011mm 0.1499mm 0.2007mm 0.1499mm 0.2007mm 0.1499mm 0.2007mm 0.1499mm 0.2007mm 0.1499mm 0.2007mm 0.1499mm 0.2007mm 0.1499mm 0.2007mm"/>
-<param name="mdWireWire" value="8mil"/>
-<param name="mdWirePad" value="8mil"/>
-<param name="mdWireVia" value="8mil"/>
+<param name="mtCopper" value="0.035mm 0.035mm 0.035mm 0.035mm 0.035mm 0.035mm 0.035mm 0.035mm 0.035mm 0.035mm 0.035mm 0.035mm 0.035mm 0.035mm 0.035mm 0.035mm"/>
+<param name="mtIsolate" value="1.5mm 0.15mm 0.2mm 0.15mm 0.2mm 0.15mm 0.2mm 0.15mm 0.2mm 0.15mm 0.2mm 0.15mm 0.2mm 0.15mm 0.2mm"/>
+<param name="mdWireWire" value="6mil"/>
+<param name="mdWirePad" value="6mil"/>
+<param name="mdWireVia" value="6mil"/>
 <param name="mdPadPad" value="6mil"/>
-<param name="mdPadVia" value="8mil"/>
-<param name="mdViaVia" value="8mil"/>
+<param name="mdPadVia" value="6mil"/>
+<param name="mdViaVia" value="6mil"/>
 <param name="mdSmdPad" value="6mil"/>
 <param name="mdSmdVia" value="6mil"/>
 <param name="mdSmdSmd" value="6mil"/>
-<param name="mdViaViaSameLayer" value="8mil"/>
+<param name="mdViaViaSameLayer" value="6mil"/>
 <param name="mnLayersViaInSmd" value="2"/>
-<param name="mdCopperDimension" value="15mil"/>
-<param name="mdDrill" value="8mil"/>
+<param name="mdCopperDimension" value="40mil"/>
+<param name="mdDrill" value="6mil"/>
 <param name="mdSmdStop" value="0mil"/>
-<param name="msWidth" value="8mil"/>
-<param name="msDrill" value="13mil"/>
-<param name="msMicroVia" value="13mil"/>
+<param name="msWidth" value="6mil"/>
+<param name="msDrill" value="0.35mm"/>
+<param name="msMicroVia" value="9.99mm"/>
 <param name="msBlindViaRatio" value="0.5"/>
 <param name="rvPadTop" value="0.25"/>
@@
 <param name="rvMicroViaOuter" value="0.25"/>
 <param name="rvMicroViaInner" value="0.25"/>
-<param name="rlMinPadTop" value="7mil"/>
+<param name="rlMinPadTop" value="10mil"/>
 <param name="rlMaxPadTop" value="20mil"/>
-<param name="rlMinPadInner" value="7mil"/>
+<param name="rlMinPadInner" value="10mil"/>
 <param name="rlMaxPadInner" value="20mil"/>
-<param name="rlMinPadBottom" value="7mil"/>
+<param name="rlMinPadBottom" value="10mil"/>
 <param name="rlMaxPadBottom" value="20mil"/>
-<param name="rlMinViaOuter" value="7mil"/>
+<param name="rlMinViaOuter" value="8mil"/>
 <param name="rlMaxViaOuter" value="20mil"/>
-<param name="rlMinViaInner" value="7mil"/>
+<param name="rlMinViaInner" value="8mil"/>
 <param name="rlMaxViaInner" value="20mil"/>
 <param name="rlMinMicroViaOuter" value="4mil"/>
@@
 <param name="mvStopFrame" value="1"/>
 <param name="mvCreamFrame" value="0"/>
-<param name="mlMinStopFrame" value="3mil"/>
-<param name="mlMaxStopFrame" value="3mil"/>
+<param name="mlMinStopFrame" value="4mil"/>
+<param name="mlMaxStopFrame" value="4mil"/>
 <param name="mlMinCreamFrame" value="0mil"/>
 <param name="mlMaxCreamFrame" value="0mil"/>
@@
 <via x="4.445" y="16.383" extent="1-16" drill="0.6"/>
 <wire x1="25.4" y1="38.52" x2="25.4" y2="38.354" width="0.4064" layer="1"/>
-<wire x1="25.4" y1="38.354" x2="25.4" y2="37.084" width="0.4064" layer="1"/>
+<wire x1="25.4" y1="38.354" x2="25.4" y2="37.084" width="0.762" layer="1"/>
 <via x="25.4" y="37.084" extent="1-16" drill="0.6"/>
-<wire x1="21.209" y1="38.52" x2="21.209" y2="37.084" width="0.4064" layer="1"/>
+<wire x1="21.209" y1="38.52" x2="21.209" y2="37.084" width="0.762" layer="1"/>
 <via x="21.209" y="37.084" extent="1-16" drill="0.6"/>
 <wire x1="24.384" y1="42.832" x2="24.257" y2="42.705" width="0.508" layer="1"/>
@@
 <contactref element="CB" pad="1"/>
 <contactref element="U1" pad="3"/>
-<wire x1="23.114" y1="42.832" x2="23.114" y2="40.22" width="0.508" layer="1"/>
+<wire x1="23.114" y1="42.832" x2="23.114" y2="40.22" width="0.762" layer="1"/>
 </signal>
 <signal name="FB">
@@
 <contactref element="RFB2" pad="1"/>
 <contactref element="U1" pad="6"/>
-<wire x1="25.4" y1="40.22" x2="27.305" y2="40.22" width="0.508" layer="1"/>
-<wire x1="26.924" y1="42.832" x2="27.11576875" y2="42.64023125" width="0.508" layer="1"/>
-<wire x1="27.305" y1="40.22" x2="27.11576875" y2="40.40923125" width="0.508" layer="1"/>
-<wire x1="27.11576875" y1="42.64023125" x2="27.11576875" y2="40.40923125" width="0.508" layer="1"/>
+<wire x1="25.4" y1="40.22" x2="27.305" y2="40.22" width="0.762" layer="1"/>
+<wire x1="26.924" y1="42.832" x2="26.98876875" y2="42.76723125" width="0.508" layer="1"/>
+<wire x1="27.305" y1="40.22" x2="26.98876875" y2="40.53623125" width="0.508" layer="1"/>
+<wire x1="26.98876875" y1="42.76723125" x2="26.98876875" y2="40.53623125" width="0.762" layer="1"/>
 </signal>
 <signal name="CUTOUT5">
