File: X14-Conversion.brd (EAGLE design)
At the start: 50.8 x 62.9 mm, 22 parts, among them U1 BUCK,LM2678S-ADJ

Commit message: add 1x2 headers to board
Parts:
- added 3.3V_H, 5.2V_H, GND_H: (no value), SparkFun-Connectors:1X02
- moved U$2 0.25 mm to (46.0, 16.5)
- moved U$7 0.25 mm to (46.0, 31.0)
Connections:
- net 3.3V: now also 3.3V_H.1, 3.3V_H.2
- net 5.2V: now also 5.2V_H.1, 5.2V_H.2
- net GND: now also GND_H.1, GND_H.2
Routing:
- net 5.2V: track 0.00 -> 29.9 mm
- net 3.3V: track 27.2 -> 49.3 mm
- net GND: vias 10 -> 17
- net 12V: vias 0 -> 4
Changed lines of the file:
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@@
 <text x="44.45" y="38.1" size="1.27" layer="21">12V</text>
 <text x="22.733" y="14.478" size="1.27" layer="21">5.2V</text>
-<text x="43.815" y="20.32" size="1.27" layer="21">3.3V</text>
-<text x="43.688" y="26.035" size="1.27" layer="21">GND</text>
+<text x="44.069" y="20.32" size="1.27" layer="21">3.3V</text>
+<text x="43.942" y="26.035" size="1.27" layer="21">GND</text>
 <text x="3.175" y="14.859" size="1.27" layer="21">GND</text>
 <text x="28.575" y="58.674" size="1.27" layer="21">GND</text>
@@
 1/7/2022
 </text>
+<text x="2.794" y="25.908" size="1.27" layer="21" rot="R90">GND</text>
+<text x="2.794" y="35.56" size="1.27" layer="21" rot="R90">3.3V</text>
+<text x="2.794" y="44.958" size="1.27" layer="21" rot="R90">5.2V</text>
 </plain>
 <attributes>
@@
 <attribute name="VALUE" x="12.556209375" y="16.4333" size="0.508" layer="27" rot="R180"/>
 </element>
-<element name="U$2" library="testpoints" package="3.3V_TESTPOINT" value="3.3V_TESTPOINT" x="45.72" y="16.51" smashed="yes"/>
+<element name="U$2" library="testpoints" package="3.3V_TESTPOINT" value="3.3V_TESTPOINT" x="45.974" y="16.51" smashed="yes"/>
 <element name="U$3" library="testpoints" package="5.2V_TESTPOINT" value="5.2V_TESTPOINT" x="24.384" y="10.668" smashed="yes"/>
 <element name="U$4" library="testpoints" package="12V_TESTPOINT" value="12V_TESTPOINT" x="45.974" y="42.672" smashed="yes"/>
 <element name="U$5" library="testpoints" package="GND_TESTPOINT" value="GND_TESTPOINT" x="30.607" y="63.627" smashed="yes"/>
 <element name="U$6" library="testpoints" package="GND_TESTPOINT" value="GND_TESTPOINT" x="5.08" y="11.049" smashed="yes"/>
-<element name="U$7" library="testpoints" package="GND_TESTPOINT" value="GND_TESTPOINT" x="45.72" y="30.988" smashed="yes"/>
+<element name="U$7" library="testpoints" package="GND_TESTPOINT" value="GND_TESTPOINT" x="45.974" y="30.988" smashed="yes"/>
 <element name="RFB2" library="SparkFun-Resistors" library_urn="urn:adsk.eagle:library:532" package="0603" package3d_urn="urn:adsk.eagle:package:39650/1" value="3.32kΩ" x="27.305" y="39.37" smashed="yes" rot="R270">
 <attribute name="NAME" x="27.43835" y="37.28085" size="0.508" layer="25" ratio="20" align="bottom-center"/>
@@
 <attribute name="NAME" x="33.528" y="22.479" size="0.762" layer="25" rot="R90" align="bottom-center"/>
 <attribute name="VALUE" x="27.559" y="19.939" size="1.27" layer="27" align="top-center" display="off"/>
+</element>
+<element name="3.3V_H" library="SparkFun-Connectors" library_urn="urn:adsk.eagle:library:513" package="1X02" package3d_urn="urn:adsk.eagle:package:38039/1" value="" x="4.572" y="36.068" smashed="yes" rot="R90">
+<attribute name="NAME" x="3.175" y="34.798" size="0.6096" layer="25" ratio="20" rot="R90" display="off"/>
+<attribute name="VALUE" x="6.604" y="34.798" size="0.6096" layer="27" font="vector" ratio="20" rot="R90"/>
+</element>
+<element name="5.2V_H" library="SparkFun-Connectors" library_urn="urn:adsk.eagle:library:513" package="1X02" package3d_urn="urn:adsk.eagle:package:38039/1" value="" x="4.572" y="45.466" smashed="yes" rot="R90">
+<attribute name="NAME" x="3.175" y="44.196" size="0.6096" layer="25" ratio="20" rot="R90" display="off"/>
+<attribute name="VALUE" x="6.604" y="44.196" size="0.6096" layer="27" font="vector" ratio="20" rot="R90"/>
+</element>
+<element name="GND_H" library="SparkFun-Connectors" library_urn="urn:adsk.eagle:library:513" package="1X02" package3d_urn="urn:adsk.eagle:package:38039/1" value="" x="4.572" y="26.67" smashed="yes" rot="R90">
+<attribute name="NAME" x="3.175" y="25.4" size="0.6096" layer="25" ratio="20" rot="R90" display="off"/>
+<attribute name="VALUE" x="6.604" y="25.4" size="0.6096" layer="27" font="vector" ratio="20" rot="R90"/>
 </element>
 </elements>
@@
 <contactref element="U1" pad="8"/>
 <contactref element="U1" pad="4"/>
-<via x="40.894" y="34.544" extent="1-16" drill="0.6"/>
-<via x="40.894" y="30.988" extent="1-16" drill="0.6"/>
-<via x="40.894" y="24.638" extent="1-16" drill="0.6"/>
-<via x="46.736" y="24.638" extent="1-16" drill="0.6"/>
+<via x="39.878" y="34.036" extent="1-16" drill="0.6"/>
+<via x="39.878" y="29.718" extent="1-16" drill="0.6"/>
+<via x="39.878" y="25.4" extent="1-16" drill="0.6"/>
 <contactref element="COUT1" pad="-"/>
 <contactref element="COUT2" pad="-"/>
 <contactref element="COUT3" pad="-"/>
 <via x="47.371" y="50.165" extent="1-16" drill="0.6"/>
-<via x="34.798" y="34.544" extent="1-16" drill="0.6"/>
-<via x="34.798" y="30.988" extent="1-16" drill="0.6"/>
-<via x="34.798" y="24.384" extent="1-16" drill="0.6"/>
+<via x="35.56" y="34.036" extent="1-16" drill="0.6"/>
+<via x="35.56" y="29.718" extent="1-16" drill="0.6"/>
+<via x="35.56" y="25.4" extent="1-16" drill="0.6"/>
 <wire x1="25.4" y1="38.52" x2="25.4" y2="38.354" width="0.4064" layer="1"/>
 <wire x1="25.4" y1="38.354" x2="25.4" y2="37.084" width="0.762" layer="1"/>
@@
 <wire x1="24.257" y1="42.705" x2="24.257" y2="39.497" width="0.508" layer="1"/>
 <wire x1="24.257" y1="39.497" x2="25.4" y2="38.354" width="0.508" layer="1"/>
+<contactref element="GND_H" pad="2"/>
+<contactref element="GND_H" pad="1"/>
+<via x="15.494" y="13.208" extent="1-16" drill="0.6"/>
+<via x="15.494" y="8.89" extent="1-16" drill="0.6"/>
+<via x="11.176" y="13.208" extent="1-16" drill="0.6"/>
+<via x="11.176" y="8.89" extent="1-16" drill="0.6"/>
+<via x="23.622" y="65.786" extent="1-16" drill="0.6"/>
+<via x="23.622" y="61.468" extent="1-16" drill="0.6"/>
+<via x="19.304" y="65.786" extent="1-16" drill="0.6"/>
+<via x="19.304" y="61.468" extent="1-16" drill="0.6"/>
 </signal>
 <signal name="3.3V">
@@
 <wire x1="16.3712" y1="18.1728" x2="15.0495" y2="18.1728" width="0.762" layer="1"/>
 <contactref element="AZ1117C" pad="4" route="any" routetag="G$1.OUTPUT"/>
-<via x="40.894" y="19.05" extent="1-16" drill="0.6"/>
-<via x="40.894" y="14.224" extent="1-16" drill="0.6"/>
-<via x="34.671" y="19.05" extent="1-16" drill="0.6"/>
-<via x="34.671" y="14.224" extent="1-16" drill="0.6"/>
+<via x="39.878" y="18.542" extent="1-16" drill="0.6"/>
+<via x="39.878" y="14.224" extent="1-16" drill="0.6"/>
+<via x="35.433" y="18.542" extent="1-16" drill="0.6"/>
+<via x="35.433" y="14.224" extent="1-16" drill="0.6"/>
 <polygon width="0.508" layer="16" isolate="0.3048">
 <vertex x="45.8089" y="20.59305"/>
@@
 </polygon>
 <wire x1="9.525" y1="19.304" x2="12.8284" y2="19.304" width="0.762" layer="1"/>
-<wire x1="16.383" y1="18.161" x2="30.734" y2="18.161" width="0.762" layer="16"/>
-<wire x1="30.734" y1="18.161" x2="34.671" y2="14.224" width="0.762" layer="16"/>
+<wire x1="16.383" y1="18.161" x2="31.496" y2="18.161" width="0.762" layer="16"/>
+<wire x1="31.496" y1="18.161" x2="35.433" y2="14.224" width="0.762" layer="16"/>
+<contactref element="3.3V_H" pad="2"/>
+<contactref element="3.3V_H" pad="1"/>
+<wire x1="4.572" y1="36.068" x2="6.985" y2="33.655" width="0.508" layer="1"/>
+<wire x1="6.985" y1="33.655" x2="6.985" y2="21.844" width="0.508" layer="1"/>
+<wire x1="6.985" y1="21.844" x2="9.525" y2="19.304" width="0.508" layer="1"/>
+<wire x1="4.572" y1="36.068" x2="4.572" y2="38.608" width="0.508" layer="1"/>
 </signal>
 <signal name="5.2V">
@@
 <vertex x="28.7655" y="17.2212"/>
 </polygon>
+<contactref element="5.2V_H" pad="2"/>
+<contactref element="5.2V_H" pad="1"/>
+<wire x1="4.572" y1="45.466" x2="4.572" y2="48.006" width="0.508" layer="1"/>
+<wire x1="4.572" y1="45.466" x2="8.0822" y2="41.9558" width="0.508" layer="1"/>
+<wire x1="8.0822" y1="41.9558" x2="8.0822" y2="27.7318" width="0.508" layer="1"/>
+<wire x1="14.986" y1="24.626" x2="11.188" y2="24.626" width="0.508" layer="1"/>
+<wire x1="11.188" y1="24.626" x2="8.0822" y2="27.7318" width="0.508" layer="1"/>
 </signal>
 <signal name="12V">
@@
 <vertex x="13.7541" y="44.7929"/>
 </polygon>
+<via x="39.878" y="45.466" extent="1-16" drill="0.6"/>
+<via x="39.878" y="41.148" extent="1-16" drill="0.6"/>
+<via x="35.56" y="45.466" extent="1-16" drill="0.6"/>
+<via x="35.56" y="41.148" extent="1-16" drill="0.6"/>
 </signal>
 <signal name="SW">

Commit message: Update X14-Conversion.brd
Parts:
- moved U$3 0.25 mm to (24.4, 10.9)
- moved U$6 0.13 mm to (5.09, 10.9)
Changed lines of the file:
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@@
 <wire x1="35.56" y1="53.34" x2="50.8" y2="53.34" width="0" layer="20"/>
 <text x="44.45" y="38.1" size="1.27" layer="21">12V</text>
-<text x="22.733" y="14.478" size="1.27" layer="21">5.2V</text>
+<text x="22.733" y="14.732" size="1.27" layer="21">5.2V</text>
 <text x="44.069" y="20.32" size="1.27" layer="21">3.3V</text>
 <text x="43.942" y="26.035" size="1.27" layer="21">GND</text>
@@
 </element>
 <element name="U$2" library="testpoints" package="3.3V_TESTPOINT" value="3.3V_TESTPOINT" x="45.974" y="16.51" smashed="yes"/>
-<element name="U$3" library="testpoints" package="5.2V_TESTPOINT" value="5.2V_TESTPOINT" x="24.384" y="10.668" smashed="yes"/>
+<element name="U$3" library="testpoints" package="5.2V_TESTPOINT" value="5.2V_TESTPOINT" x="24.384" y="10.922" smashed="yes"/>
 <element name="U$4" library="testpoints" package="12V_TESTPOINT" value="12V_TESTPOINT" x="45.974" y="42.672" smashed="yes"/>
 <element name="U$5" library="testpoints" package="GND_TESTPOINT" value="GND_TESTPOINT" x="30.607" y="63.627" smashed="yes"/>
-<element name="U$6" library="testpoints" package="GND_TESTPOINT" value="GND_TESTPOINT" x="5.08" y="11.049" smashed="yes"/>
+<element name="U$6" library="testpoints" package="GND_TESTPOINT" value="GND_TESTPOINT" x="5.08635" y="10.91565" smashed="yes"/>
 <element name="U$7" library="testpoints" package="GND_TESTPOINT" value="GND_TESTPOINT" x="45.974" y="30.988" smashed="yes"/>
 <element name="RFB2" library="SparkFun-Resistors" library_urn="urn:adsk.eagle:library:532" package="0603" package3d_urn="urn:adsk.eagle:package:39650/1" value="3.32kΩ" x="27.305" y="39.37" smashed="yes" rot="R270">
